Commit message: base_link

File: drive/urdf/drive.urdf (robot description, URDF)
Before this commit: robot drive, 15 links, 14 joints
Links:
- removed link base
- added link base_link, mass 12.720238406316; collision mesh filename=package://drive/meshes/base.STL; visual mesh filename=package://drive/meshes/base.STL
Joints:
- joint bogie_front_left_joint: parent base -> base_link
- joint bogie_front_right_joint: parent base -> base_link
- joint bogie_middle_left_joint: parent base -> base_link
- joint bogie_middle_right_joint: parent base -> base_link
- joint imu_joint: parent base -> base_link
- joint lidar_joint: parent base -> base_link
- joint rocker_left_joint: parent base -> base_link
- joint rocker_right_joint: parent base -> base_link
