Commit message: gazebo issue

File: drive/models/drive/urdf/drive.urdf (robot description, URDF)
Before this commit: robot drive, 15 links, 14 joints
Links:
- link base_link: geometry collision mesh filename=package://drive/meshes/base.stl; visual mesh filename=package://drive/meshes/base.stl
- link bogie_front_left: geometry collision mesh filename=package://drive/meshes/bogie_front_left.stl; visual mesh filename=package://drive/meshes/bogie_front_left.stl
- link bogie_front_right: geometry collision mesh filename=package://drive/meshes/bogie_front_right.stl; visual mesh filename=package://drive/meshes/bogie_front_right.stl
- link bogie_middle_left: geometry collision mesh filename=package://drive/meshes/bogie_middle_left.stl; visual mesh filename=package://drive/meshes/bogie_middle_left.stl
- link bogie_middle_right: geometry collision mesh filename=package://drive/meshes/bogie_middle_right.stl; visual mesh filename=package://drive/meshes/bogie_middle_right.stl
- link lidar_link: geometry collision mesh filename=package://drive/meshes/lidar.stl scale=1 1 1; visual mesh filename=package://drive/meshes/lidar.stl scale=1 1 1
- link rocker_left: geometry collision mesh filename=package://drive/meshes/rocker_left.stl; visual mesh filename=package://drive/meshes/rocker_left.stl
- link rocker_right: geometry collision mesh filename=package://drive/meshes/rocker_right.stl; visual mesh filename=package://drive/meshes/rocker_right.stl
- link wheel_1: geometry collision mesh filename=package://drive/meshes/wheel_1.stl; visual mesh filename=package://drive/meshes/wheel_1.stl
- link wheel_2: geometry collision mesh filename=package://drive/meshes/wheel_2.stl; visual mesh filename=package://drive/meshes/wheel_2.stl
- link wheel_3: geometry collision mesh filename=package://drive/meshes/wheel_3.stl; visual mesh filename=package://drive/meshes/wheel_3.stl
- link wheel_4: geometry collision mesh filename=package://drive/meshes/wheel_4.stl; visual mesh filename=package://drive/meshes/wheel_4.stl
- link wheel_5: geometry collision mesh filename=package://drive/meshes/wheel_5.stl; visual mesh filename=package://drive/meshes/wheel_5.stl
- link wheel_6: geometry collision mesh filename=package://drive/meshes/wheel_6.stl; visual mesh filename=package://drive/meshes/wheel_6.stl

Commit message: lidar fix

File: drive/models/drive/urdf/drive.urdf (robot description, URDF)
Before this commit: robot drive, 15 links, 14 joints
Links:
- removed link lidar_link
- added link lidar, mass 0.5; collision cylinder length=0.1 radius=0.05; visual cylinder length=0.1 radius=0.05
Joints:
- joint lidar_joint: child lidar_link -> lidar; origin xyz=0.3 0 0.2 rpy=0 0 0 -> xyz=0 0 0.3 rpy=0 0 0

Commit message: damping

File: drive/models/drive/urdf/drive.urdf (robot description, URDF)
Before this commit: robot drive, 15 links, 14 joints
Links:
- link wheel_1: geometry collision cylinder length=0.04 radius=0.06; visual mesh filename=package://drive/meshes/wheel_1.stl
- link wheel_2: geometry collision cylinder length=0.04 radius=0.06; visual mesh filename=package://drive/meshes/wheel_2.stl
- link wheel_3: geometry collision cylinder length=0.04 radius=0.06; visual mesh filename=package://drive/meshes/wheel_3.stl
- link wheel_4: geometry collision cylinder length=0.04 radius=0.06; visual mesh filename=package://drive/meshes/wheel_4.stl
- link wheel_5: geometry collision cylinder length=0.04 radius=0.06; visual mesh filename=package://drive/meshes/wheel_5.stl
- link wheel_6: geometry collision cylinder length=0.04 radius=0.06; visual mesh filename=package://drive/meshes/wheel_6.stl

Commit message: balanced

File: drive/models/drive/urdf/drive.urdf (robot description, URDF)
Before this commit: robot drive, 15 links, 14 joints
Links:
- link base_link: mass 12.720238406316 -> 1
